Commit message: closing the gap between two arms

File: dual_arm_panda_moveit_config/config/panda.urdf.xacro (robot description, xacro)
@@ -15,5 +15,5 @@
         parent="world"
         initial_positions_file="$(arg left_initial_positions_file)">
-        <origin xyz="0 -1.5 0" rpy="0 0 0" />
+        <origin xyz="0 -0.25 0" rpy="0 0 0" />
     </xacro:panda_arm>
     <!-- Right arm -->
@@ -23,5 +23,5 @@
         parent="world"
         initial_positions_file="$(arg right_initial_positions_file)">
-        <origin xyz="0 1.5 0" rpy="0 0 0" />
+        <origin xyz="0 0.25 0" rpy="0 0 0" />
     </xacro:panda_arm>
 </robot>
